File: hardware/BlueBus.sch (EAGLE design)
At the start: 130 parts, among them Q1 NMOSFET-BSS138K, Q2 PMOSFET-DMP32D4S, Q3 NMOSFET-BSS138K, X1 CRYSTAL-12MHZ

Commit message: [IMP] hardware: v1.5 High Voltage improvements * Remove XRP6759 * Remove Old Tantalum C1 * Remove V1 * Remove L1 * Add common mode choke at input (L1) to filter out A/C * Add new Aluminum Polymer input Capacitor rated for 35v (C1) * Add MPQ4420 wide input voltage switching regulator for 12v -> 5v regulation * Add XC6702 to protect Q2 from trancients and provide a constant voltage to TEL ON and Microphone power * Power Microphone through 12v rail * Rewire 3.3v net * Rewire 5v net * Fix decoupling cap positioning for PIC24
Parts:
- removed D2: 2A/100V, Passives:SCHOTTKYDIODE2A30V
- removed F2: 0468.500NR, Passives:0468.500NR
- removed V1: V18AUMLA1812H, Passives:V18AUMLA1812H
- removed XRP7659: XRP7659SOT23-6, ICs:XRP7659SOT23-6
- added C50: 2.2uF, Passives:2.2UF
- added C51, C54, C56: 10uF, Passives:10UF2012
- added C52, C53, C55: 0.1uF, Passives:0.1UF
- added L2: ETQ-P4M100KFN, Passives:ETQ-P4M100KFN
- added MPQ4420: MPQ4420, ICs:MPQ4420
- added R36: 18k, Passives:18KOHM
- added R37, R38: 100, Passives:100OHM
- added XC6702: XC6702DC018PR-G, ICs:XC6702DC018PR-G
- C1: value 100uF -> RHS1V101MCN1GS; device Passives:100UF2917 -> Passives:RHS1V101MCN1GS
- C10, C11: value 0.1uF -> 10uF; device Passives:0.1UF -> Passives:10UF
- C12: value 0.1uF -> 1uF; device Passives:0.1UF -> Passives:1UF
- C13, C44: value 10uF -> 1uF; device Passives:10UF2012 -> Passives:1UF
- C14: value 47nF -> 0.1uF; device Passives:47NF -> Passives:0.1UF
- C15: value 2.2uF -> 0.1uF; device Passives:2.2UF -> Passives:0.1UF
- C16: value 0.0001UF -> 0.1uF; device Passives:0.0001UF -> Passives:0.1UF
- C18, C29: value 10uF -> 0.1uF; device Passives:10UF2012 -> Passives:0.1UF
- C19, C41: value 0.1uF -> 10uF; device Passives:0.1UF -> Passives:10UF2012
- C2: value 0.01uF -> 22uF; device Passives:0.01UF -> Passives:22UF
- C21: value 4.7uF -> 2.2uF; device Passives:4.7UF -> Passives:2.2UF
- C22: value 0.1uF -> 0.0001UF; device Passives:0.1UF -> Passives:0.0001UF
- C23: value 0.1uF -> 47nF; device Passives:0.1UF -> Passives:47NF
- C24, C25: value 20pF -> 0.1uF; device Passives:20PF -> Passives:0.1UF
- C26: value 1uF -> 10uF; device Passives:1UF -> Passives:10UF2012
- C28: value 47UF -> 4.7uF; device Passives:47UF -> Passives:4.7UF
- C3: value 10uF -> 22uF; device Passives:10UF2012 -> Passives:22UF
- C30, C34: value 1uF -> 0.1uF; device Passives:1UF -> Passives:0.1UF
- C31, C32: value 1uF -> 20pF; device Passives:1UF -> Passives:20PF
- C35: value 10uF -> 47UF; device Passives:10UF2012 -> Passives:47UF
- C36: value 220pF -> 1uF; device Passives:220PF -> Passives:1UF
- C37: value 220pF -> 10uF; device Passives:220PF -> Passives:10UF2012
- C38: value 9nF -> 1uF; device Passives:9NF -> Passives:1UF
- C39: value 9nF -> 220pF; device Passives:9NF -> Passives:220PF
- C4: value 22uF -> 0.1uF; device Passives:22UF -> Passives:0.1UF
- C40: value 10uF -> 220pF; device Passives:10UF2012 -> Passives:220PF
- C42, C43: value 2.2uF -> 1uF; device Passives:2.2UF -> Passives:1UF
- C45, C46: value 0.1uF -> 10nF; device Passives:0.1UF -> Passives:10NF
- C49: value 10uF -> 2.2uF; device Passives:10UF2012 -> Passives:2.2UF
- C5: value 1uF -> 2.2uF; device Passives:1UF -> Passives:2.2UF
- D1, D3: device Passives:SCHOTTKYDIODE2A30V -> Passives:SCHOTTKYDIODE2A100V
- L1: value 4.7uH -> ACM70V-701-2PL-TL00; device Passives:MPLCG0630L4R7 -> Passives:ACM70V-701-2PL-TL00
- R10: value 10k -> 41.2KOHM; device Passives:10KOHM -> Passives:41.2KOHM
- R11: value 10 -> 4.7k; device Passives:10OHM -> Passives:4.7KOHM
- R12: value 10k -> 210; device Passives:10KOHM -> Passives:210OHM
- R14: value 100k -> 10; device Passives:100KOHM -> Passives:10OHM
- R15: value 100k -> 10k; device Passives:100KOHM -> Passives:10KOHM
- R16, R18: value 2k -> 100k; device Passives:2KOHM -> Passives:100KOHM
- R17: value 2k -> 10k; device Passives:2KOHM -> Passives:10KOHM
- R19: value 2 -> 2k; device Passives:2OHM -> Passives:2KOHM
- R20, R21: value 10k -> 2k; device Passives:10KOHM -> Passives:2KOHM
- R22: value 10k -> 2; device Passives:10KOHM -> Passives:2OHM
- R24: value 210 -> 10k; device Passives:210OHM -> Passives:10KOHM
- R25: value 110 -> 10k; device Passives:110OHM -> Passives:10KOHM
- R26: value 75 -> 10k; device Passives:75OHM -> Passives:10KOHM
- R27: value 10k -> 110; device Passives:10KOHM -> Passives:110OHM
- R28: value 4.7k -> 210; device Passives:4.7KOHM -> Passives:210OHM
- R33: value 18k -> 10k; device Passives:18KOHM -> Passives:10KOHM
- R34: value 110 -> 75; device Passives:110OHM -> Passives:75OHM
- R35: value 110 -> 4.7k; device Passives:110OHM -> Passives:4.7KOHM
- R5: value 9.09k -> 100k; device Passives:9.09KOHM -> Passives:100KOHM
- R6: value 47k -> 100k; device Passives:47KOHM -> Passives:100KOHM
- R7: value 100k -> 20OHM; device Passives:100KOHM -> Passives:20OHM
- R8: value 4.7k -> 51KOHM; device Passives:4.7KOHM -> Passives:51KOHM
- R9: value 210 -> 7.68KOHM; device Passives:210OHM -> Passives:7.68KOHM
Connections:
- net 12V_VIN renamed VBAT
- net VIN_DIODE renamed VBAT_DIODE
- removed net RAW_3.3V: C6.1, F2.IN, XC6210.VOUT
- new net 12V: C5.1, Q2.S, R3.2, R35.1, XC6702.VOUT
- new net 5VREG_BS_CAP: C8.1, R7.2
- new net 5VREG_FB_T: R10.1, R8.1, R9.2
- new net 5VREG_PG: MPQ4420.PG, R5.1
- new net 5VREG_VCC: C7.1, MPQ4420.VCC, R5.2
- new net VBAT_FUSE: F1.IN, L1.1
- net 3.3V: now also C12.1, C14.1, C15.2, C16.2, C17.2, C20.2, C24.1, C30.1, C33.1, C48.1, C51.1, C52.1, C53.1, C54.1, R11.2, R16.2, R17.1, R21.2, R24.2, R26.2, R29.1, R32.1, XC6210.VOUT; no longer C10.2, C11.2, C20.1, C23.1, C26.1, C40.1, C41.1, C44.1, C45.1, C46.1, C7.1, C8.2, C9.2, F2.OUT, R10.1, R12.2, R14.2, R17.2, R19.2, R28.1, R31.1, R8.2
- net 5V: now also C13.1, C2.1, C25.1, C26.1, C3.1, C36.1, C37.1, C38.1, C41.1, C42.1, L2.2, R10.2; no longer C17.1, C18.1, C29.1, C30.1, C31.1, C34.1, C35.1, C5.1, L1.2, R32.1, R6.2
- net 5VREG_BS: now also MPQ4420.BS, R7.1; no longer C2.1, XRP7659.BS
- net 5VREG_EN: now also MPQ4420.EN, R6.1; no longer R7.2, XRP7659.EN
- net 5VREG_FB: now also MPQ4420.FB, R8.2; no longer R5.1, R6.1, XRP7659.FB
- net 5VREG_SW: now also C8.2, L2.1, MPQ4420.SW; no longer C2.2, D2.C, L1.1, XRP7659.SW
- net AGND: now also C46.2, C47.2, C48.2, C49.1, C51.2, C52.2; no longer C38.2, C39.2, C40.2, C41.2, C42.1, C44.2
- net BT_3V3_FILTER: now also C28.1, R22.1; no longer C21.1, R19.1
- net BT_DOUT: now also C34.2, R34.2; no longer C27.2, R26.2
- net BT_MIC_L: now also C35.1; no longer C28.1
- net BT_RST: now also R24.1; no longer R22.1
- net BT_URX: now also R25.1; no longer R21.1
- net BT_URX_RES: now also R25.2; no longer R21.2
- net BT_UTX: now also R26.1; no longer R20.1
- net DAC_CAPM: now also C50.2; no longer C43.2
- net DAC_CAPP: now also C50.1; no longer C43.1
- net DAC_LDOO: now also C55.1, C56.1; no longer C48.1, C49.1
- net DAC_OUT_L: now also R38.1; no longer R34.1
- net DAC_OUT_R: now also R37.1; no longer R35.1
- net DAC_VNEG: now also C49.2; no longer C42.2
- net EE_CS: now also R11.1; no longer R8.1
- net GND: now also C10.2, C11.2, C16.1, C17.1, C2.2, C20.1, C21.1, C22.2, C27.2, C28.2, C33.2, C38.2, C39.2, C40.2, C41.2, C42.2, C44.2, C53.2, C54.2, C55.2, C56.2, C9.2, L1.2, L1.3, MPQ4420.GND, R31.1, R33.1, R34.1, R4.1, R9.1, XC6702.GND; no longer C10.1, C11.1, C16.2, C17.2, C20.2, C21.2, C29.2, C34.2, C35.2, C46.2, C47.2, C48.2, C49.2, C8.1, C9.1, D2.A, R25.1, R26.1, R29.1, R3.1, R5.2, V1.IN, XRP7659.GND
- net IBUS: now also R14.1; no longer R11.1
- net IBUS_5V: now also C21.2, R6.2; no longer C15.2, R7.1
- net IBUS_FILT: now also C22.1, R14.2; no longer C16.1, R11.2
- net MCU_MCLR: now also R12.2; no longer R9.2
- net MCU_MCLR_RES: now also C18.1, R12.1, R13.2; no longer C12.1, R10.2, R9.1
- net MCU_ON_LED: now also R19.2; no longer R16.2
- net MCU_ON_LED_RES: now also R19.1; no longer R16.1
- net MCU_RECOV: now also R15.1; no longer R12.1
- net MCU_SCK3: now also R32.2; no longer R28.2
- net MCU_TEL_ON: now also R4.2; no longer R3.2
- net MCU_URX: now also R16.1; no longer R14.1
- net MCU_UTX: now also R18.1; no longer R15.1
- net MCU_VCAP: now also C19.1; no longer C13.1
- net RX_LED_RES: now also R20.1; no longer R17.1
- net SPDIF_OUT: now also C29.1; no longer C22.1
- net SPDIF_RX: now also C34.1; no longer C27.1
- net SPKR_OUT_L: now also C46.1, R38.2; no longer C38.1, R34.2
- net SPKR_OUT_R: now also C45.1, R37.2; no longer C39.1, R35.2
- net SYS_3V3: now also C27.1; no longer C19.1
- net SYS_UART_SEL: now also R17.2; no longer R13.2
- net TEL_AMP_IN: now also C43.1; no longer C33.1
- net TEL_AMP_INL: now also R36.2; no longer R33.2
- net TEL_AMP_INL_CAP_RES: now also C43.2, R36.1; no longer C33.2, R33.1
- net TEL_AMP_VREF: now also C44.1; no longer C32.1
- net TEL_MIC_L_OUT: now also C35.2, R35.2; no longer C28.2, R32.2
- net TEL_ON_EN: now also R3.1; no longer R4.1
- net TEL_OUT_L+: now also C39.1; no longer C37.1
- net TEL_OUT_L-: now also C40.1; no longer C36.1
- net TX_LED_RES: now also R21.1; no longer R18.1
- net VIN: now also C10.1, C11.1, C23.1, C6.1, C9.1, L1.4, MPQ4420.IN, XC6702.CE, XC6702.VIN; no longer C14.1, C3.1, F1.IN, Q2.S, R4.2, V1.OUT, XRP7659.VIN
- net WM_CSB: now also R33.2; no longer R27.2
- net WM_GPO0: now also R31.2; no longer R29.2
- net WM_RESETB: now also R29.2; no longer R31.2
- net WM_SPDIF_TX_RES: now also R28.2; no longer R24.2
- net WM_SPDIF_TX_RES2: now also C29.2, R27.2, R28.1; no longer C22.2, R24.1, R25.2
- net WM_XIN: now also C31.1; no longer C24.1
- net WM_XOP: now also C32.1; no longer C25.1
